File: nanobndecd_mk4.kicad_pcb (KiCad board)
At the start: 2 copper layers, 100 x 80 mm, 59 parts, among them CON1 5,5/2,1mm, J1 RJ45, J2 RJ45, J3 DB9, P1 CONN_01X16, P2 CONN_01X16, P3 CONN_02X08, P4 CONN_01X04, Q1 BS170, Q2 BS170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

Commit message: Final PCB
Routing:
- net /EXT_SDA: track 47.4 -> 101.4 mm, vias 0 -> 2
- net /EXT_SCL: track 59.6 -> 94.4 mm, vias 0 -> 2
Other:
- board text added: "Rev. 1"
- board text removed: "Rev. 2.3"
Changed lines of the file:
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@@
   (general
     (links 139)
-    (no_connects 2)
+    (no_connects 0)
     (area 78.256429 35.738999 200.308572 144.456001)
     (thickness 1.6)
     (drawings 38)
-    (tracks 485)
+    (tracks 508)
     (zones 0)
     (modules 59)
@@
     )
   )
-  (gr_text "Rev. 2.3" (at 183.134 121.666) (layer F.SilkS)
+  (gr_text "Rev. 1" (at 183.134 121.666) (layer F.SilkS)
     (effects (font (size 1.5 1.5) (thickness 0.3)))
   )
@@
   (segment (start 118.618 108.7755) (end 130.1115 97.282) (width 0.254) (layer B.Cu) (net 9))
   (segment (start 118.618 109.728) (end 118.618 108.7755) (width 0.254) (layer B.Cu) (net 9))
+  (segment (start 152.781 79.328) (end 152.781 80.264) (width 0.254) (layer F.Cu) (net 10))
+  (segment (start 144.526 110.617) (end 144.526 110.49) (width 0.254) (layer F.Cu) (net 10))
+  (segment (start 144.526 106.553) (end 144.526 110.617) (width 0.254) (layer F.Cu) (net 10))
+  (via (at 144.526 106.553) (size 1) (drill 0.5) (layers F.Cu B.Cu) (net 10))
+  (segment (start 151.13 99.949) (end 144.526 106.553) (width 0.254) (layer B.Cu) (net 10))
+  (segment (start 151.13 90.551) (end 151.13 99.949) (width 0.254) (layer B.Cu) (net 10))
+  (segment (start 151.257 90.424) (end 151.13 90.551) (width 0.254) (layer B.Cu) (net 10))
+  (via (at 151.257 90.424) (size 1) (drill 0.5) (layers F.Cu B.Cu) (net 10))
+  (segment (start 151.257 81.788) (end 151.257 90.424) (width 0.254) (layer F.Cu) (net 10))
+  (segment (start 152.781 80.264) (end 151.257 81.788) (width 0.254) (layer F.Cu) (net 10))
   (segment (start 152.781 79.328) (end 151.464 79.328) (width 0.254) (layer F.Cu) (net 10))
   (segment (start 153.777 73.68) (end 153.777 72.517) (width 0.254) (layer F.Cu) (net 10))
@@
   (segment (start 153.777 66.06) (end 155.448 64.389) (width 0.254) (layer F.Cu) (net 10))
   (segment (start 144.526 110.49) (end 141.4272 113.5888) (width 0.254) (layer F.Cu) (net 10))
+  (segment (start 141.4272 113.5888) (end 141.2748 113.5888) (width 0.254) (layer F.Cu) (net 10))
   (segment (start 141.2748 113.5888) (end 127.5588 113.5888) (width 0.254) (layer F.Cu) (net 10))
-  (segment (start 141.4272 113.5888) (end 141.2748 113.5888) (width 0.254) (layer F.Cu) (net 10))
   (segment (start 127.5588 113.5888) (end 123.698 109.728) (width 0.254) (layer F.Cu) (net 10))
   (segment (start 141.2748 113.538) (end 141.2748 113.5888) (width 0.254) (layer F.Cu) (net 10))
@@
   (segment (start 141.2748 113.538) (end 141.2748 113.5888) (width 0.254) (layer F.Cu) (net 10))
   (segment (start 150.3045 114.046) (end 146.7485 110.49) (width 0.254) (layer F.Cu) (net 10))
+  (segment (start 150.3045 115.6335) (end 150.3045 114.046) (width 0.254) (layer F.Cu) (net 10))
   (segment (start 146.7485 110.49) (end 144.526 110.49) (width 0.254) (layer F.Cu) (net 10))
-  (segment (start 150.3045 115.6335) (end 150.3045 114.046) (width 0.254) (layer F.Cu) (net 10))
   (segment (start 149.606 68.072) (end 147.955 66.421) (width 0.254) (layer F.Cu) (net 11))
   (segment (start 149.606 75.966) (end 149.606 68.072) (width 0.254) (layer F.Cu) (net 11))
@@
   (segment (start 141.986 77.49) (end 143.51 75.966) (width 0.254) (layer F.Cu) (net 12))
   (segment (start 116.078 109.728) (end 116.078 106.299) (width 0.254) (layer F.Cu) (net 12))
+  (segment (start 147.7645 115.6335) (end 147.7645 117.0305) (width 0.254) (layer F.Cu) (net 13))
+  (segment (start 156.083 81.915) (end 156.083 79.328) (width 0.254) (layer F.Cu) (net 13))
+  (segment (start 157.48 83.312) (end 156.083 81.915) (width 0.254) (layer F.Cu) (net 13))
+  (via (at 157.48 83.312) (size 1) (drill 0.5) (layers F.Cu B.Cu) (net 13))
+  (segment (start 161.544 87.376) (end 157.48 83.312) (width 0.254) (layer B.Cu) (net 13))
+  (segment (start 161.544 94.234) (end 161.544 87.376) (width 0.254) (layer B.Cu) (net 13))
+  (segment (start 161.671 94.361) (end 161.544 94.234) (width 0.254) (layer B.Cu) (net 13))
+  (via (at 161.671 94.361) (size 1) (drill 0.5) (layers F.Cu B.Cu) (net 13))
+  (segment (start 161.671 113.03) (end 161.671 94.361) (width 0.254) (layer F.Cu) (net 13))
+  (segment (start 157.353 117.348) (end 161.671 113.03) (width 0.254) (layer F.Cu) (net 13))
+  (segment (start 148.082 117.348) (end 157.353 117.348) (width 0.254) (layer F.Cu) (net 13))
+  (segment (start 147.7645 117.0305) (end 148.082 117.348) (width 0.254) (layer F.Cu) (net 13))
+  (segment (start 147.7645 115.6335) (end 147.7645 116.3955) (width 0.254) (layer F.Cu) (net 13))
   (segment (start 156.083 79.328) (end 162.607 79.328) (width 0.254) (layer F.Cu) (net 13))
+  (segment (start 162.607 79.328) (end 163.977 77.958) (width 0.254) (layer F.Cu) (net 13))
   (segment (start 163.977 77.958) (end 163.977 73.406) (width 0.254) (layer F.Cu) (net 13))
-  (segment (start 162.607 79.328) (end 163.977 77.958) (width 0.254) (layer F.Cu) (net 13))
   (segment (start 163.977 73.406) (end 163.977 69.195) (width 0.254) (layer F.Cu) (net 13))
   (segment (start 163.977 69.195) (end 164.211 68.961) (width 0.254) (layer F.Cu) (net 13))
