File: nanobndecd_mk4.sch (KiCad schematic (older format))
At the start: 55 parts, among them CON1 5,5/2,1mm, J1 RJ45, J2 RJ45, J3 DB9, P1 CONN_01X16, P2 CONN_01X16, P3 CONN_02X08, P4 CONN_01X04, Q1 BS170, Q2 BS170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

Commit message: Corrected U1 footprint
Parts:
- U1: footprint Transistors_TO-220:TO-220_Neutral123_Vertical_MountedFromLS_LargePads -> Transistors_TO-220:TO-220_Neutral123_Vertical_LargePads
Changed lines of the file:
@@
 LIBS:contrib
 LIBS:valves
-LIBS:nanobndecd_mk4-cache
 EELAYER 25 0
 EELAYER END
@@
 F 0 "U1" H 3550 1800 40  0000 C CNN
 F 1 "LM7805CT" H 3750 1800 40  0000 L CNN
-F 2 "Transistors_TO-220:TO-220_Neutral123_Vertical_MountedFromLS_LargePads" H 3750 1700 30  0000 C CIN
+F 2 "Transistors_TO-220:TO-220_Neutral123_Vertical_LargePads" H 3750 1700 30  0000 C CIN
 F 3 "" H 3750 1600 60  0000 C CNN
 	1    3750 1600
@@
 $Bitmap
 Pos 1100 10550
-Scale 1.000000
+Scale 1,000000
 Data
 89 50 4E 47 0D 0A 1A 0A 00 00 00 0D 49 48 44 52 00 00 01 5D 00 00 01 85 08 02 00 00 00 D1 87 B7
@@
 $Bitmap
 Pos 3150 10600
-Scale 1.000000
+Scale 1,000000
 Data
 89 50 4E 47 0D 0A 1A 0A 00 00 00 0D 49 48 44 52 00 00 02 48 00 00 00 AE 08 02 00 00 00 42 FE 65
@@
 60 18 E6 D8 09 E9 30 64 26 93 49 AF D7 93 24 89 30 0C 93 4A A5 72 B9 5C 2E 97 CB 64 32 82 20 10
 42 5C 29 42 CB 16 11 11 11 11 11 79 3C 65 67 D7 38 8E A3 69 DA 66 B3 91 24 49 92 E4 FF 01 AC 85
-47 67 F9 85 74 E5 00 00 00 00 49 45 4E 44 AE 42 60 82 AD
+47 67 F9 85 74 E5 00 00 00 00 49 45 4E 44 AE 42 60 82 E2
 EndData
 $EndBitmap

Commit message: Corrected P4 to pin header
Parts:
- P4: footprint Socket_Strips:Socket_Strip_Straight_1x04 -> Pin_Headers:Pin_Header_Straight_1x04
Changed lines of the file:
@@
 LIBS:contrib
 LIBS:valves
+LIBS:nanobndecd_mk4-cache
 EELAYER 25 0
 EELAYER END
@@
 60 18 E6 D8 09 E9 30 64 26 93 49 AF D7 93 24 89 30 0C 93 4A A5 72 B9 5C 2E 97 CB 64 32 82 20 10
 42 5C 29 42 CB 16 11 11 11 11 11 79 3C 65 67 D7 38 8E A3 69 DA 66 B3 91 24 49 92 E4 FF 01 AC 85
-47 67 F9 85 74 E5 00 00 00 00 49 45 4E 44 AE 42 60 82 E2
+47 67 F9 85 74 E5 00 00 00 00 49 45 4E 44 AE 42 60 82 30
 EndData
 $EndBitmap
@@
 F 0 "P4" H 11900 6600 50  0000 C CNN
 F 1 "CONN_01X04" V 12000 6350 50  0000 C CNN
-F 2 "Socket_Strips:Socket_Strip_Straight_1x04" H 11900 6350 60  0001 C CNN
+F 2 "Pin_Headers:Pin_Header_Straight_1x04" H 11900 6350 60  0001 C CNN
 F 3 "" H 11900 6350 60  0000 C CNN
 	1    11900 6350
